File: LP5012EVM/LP5012EVM.sch (KiCad schematic (older format))
At the start: 23 parts, among them J1 Conn_01x02, J2 Conn_01x02, J3 Conn_01x02, J4 OUT_ENABLE, J5 I2C ADDRESS SELECTOR, J6 ENABLE SELECTOR, J7 USB2ANY Connector, J8 VIN SELECTOR, J9 LED VSOURCE SELECTOR, U1 LP5012RUKR

Commit message: Inclusión de la versión custom que se fabricará para el proyecto final
Parts:
- C4: value 1uF -> 0.1uF
- J9: value LED VSOURCE SELECTOR -> LED SOURCE VOLTAGE SELECTOR
- U1: value LP5012RUKR -> LP5012
Changed lines of the file:
@@
 P 5200 1800
 F 0 "C4" H 5315 1846 50  0000 L CNN
-F 1 "1uF" H 5315 1755 50  0000 L CNN
+F 1 "0.1uF" H 5315 1755 50  0000 L CNN
 F 2 "" H 5238 1650 50  0001 C CNN
 F 3 "~" H 5200 1800 50  0001 C CNN
@@
 Wire Wire Line
 	4850 2450 5650 2450
-$Comp
-L LP5012_SCH:LP5012 U1
-U 1 1 5D915B7B
-P 6100 2850
-F 0 "U1" H 5800 3500 50  0000 C CNN
-F 1 "LP5012RUKR" H 6000 2100 50  0000 C CNN
-F 2 "" H 6050 3500 50  0000 C CNN
-F 3 "" H 6050 3500 50  0000 C CNN
-	1    6100 2850
-	1    0    0    -1
-$EndComp
 Wire Wire Line
 	5550 1550 5550 2350
@@
 P 3300 6000
 F 0 "J9" H 3350 5800 50  0000 C CNN
-F 1 "LED VSOURCE SELECTOR" H 3350 6226 50  0000 C CNN
+F 1 "LED SOURCE VOLTAGE SELECTOR" H 3350 6226 50  0000 C CNN
 F 2 "" H 3300 6000 50  0001 C CNN
 F 3 "~" H 3300 6000 50  0001 C CNN
@@
 U 1 1 5DAC5120
 P 6100 4650
-F 0 "TP4" H 6180 4642 50  0000 L CNN
+F 0 "TP4" H 6050 4750 50  0000 L CNN
 F 1 "Conn_01x02" H 6180 4551 50  0001 L CNN
 F 2 "" H 6100 4650 50  0001 C CNN
@@
 Wire Wire Line
 	5750 4750 5750 4900
+$Comp
+L LP5012_SCH:LP5012 U1
+U 1 1 5D99BF30
+P 6100 2850
+F 0 "U1" H 5800 3500 50  0000 C CNN
+F 1 "LP5012" H 5900 2100 50  0000 C CNN
+F 2 "" H 6050 3500 50  0000 C CNN
+F 3 "" H 6050 3500 50  0000 C CNN
+	1    6100 2850
+	1    0    0    -1
+$EndComp
 $EndSCHEMATC
