File: pcb/LP5012.kicad_pcb (KiCad board)
At the start: 2 copper layers, 16.2 x 24.5 mm, 16 parts, among them J1 Main Connector, U1 LP5012

Commit message: Depuración de archivos sobrantes y estructuración de carpetas
Se añaden carpetas doc, info y pcb.
Se limpian archivos que estaban de más.
Changed lines of the file:
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@@
     (arrow2b (pts (xy 140.1 72.55) (xy 141.226504 71.963579)))
   )
-  (gr_text A1 (at 143.8 79.7 270) (layer F.SilkS)
+  (gr_text A1 (at 143.8 79.7 90) (layer F.SilkS)
     (effects (font (size 0.8 0.8) (thickness 0.15)))
   )
-  (gr_text A0 (at 143.8 82.2 270) (layer F.SilkS)
+  (gr_text A0 (at 143.8 82.2 90) (layer F.SilkS)
     (effects (font (size 0.8 0.8) (thickness 0.15)))
   )
-  (gr_text EN (at 143.8 84.7 270) (layer F.SilkS)
+  (gr_text EN (at 143.8 84.7 90) (layer F.SilkS)
     (effects (font (size 0.8 0.8) (thickness 0.15)))
   )
-  (gr_text SDA (at 143.8 87.2 270) (layer F.SilkS)
+  (gr_text SDA (at 143.8 87.2 90) (layer F.SilkS)
     (effects (font (size 0.8 0.8) (thickness 0.15)))
   )
-  (gr_text SCL (at 143.8 89.8 270) (layer F.SilkS)
+  (gr_text SCL (at 143.8 89.8 90) (layer F.SilkS)
     (effects (font (size 0.8 0.8) (thickness 0.15)))
   )
-  (gr_text GND (at 143.8 92.3 270) (layer F.SilkS)
+  (gr_text GND (at 143.8 92.3 90) (layer F.SilkS)
     (effects (font (size 0.8 0.8) (thickness 0.15)))
   )
-  (gr_text 3V3 (at 143.7 94.9 270) (layer F.SilkS)
+  (gr_text 3V3 (at 143.7 94.9 90) (layer F.SilkS)
     (effects (font (size 0.8 0.8) (thickness 0.15)))
   )
@@
   (via (at 149.7 77.7) (size 1) (drill 0.5) (layers F.Cu B.Cu) (net 3))
   (via (at 155.4 77.8) (size 1) (drill 0.5) (layers F.Cu B.Cu) (net 3))
-  (via (at 155.199998 98.5) (size 1) (drill 0.4) (layers F.Cu B.Cu) (net 3))
+  (via (at 155.199998 98.5) (size 1) (drill 0.5) (layers F.Cu B.Cu) (net 3))
   (segment (start 141.7 94.9) (end 141.2 95.4) (width 0.8) (layer B.Cu) (net 3))
   (segment (start 141.2 95.4) (end 141.2 98) (width 0.8) (layer B.Cu) (net 3))

Commit message: Inclusión de modelos 3D y modificación de algunas liberías
Parts:
- D7, D8: footprint LED_SMD:LED_RGB_1210 -> LED_RGB_1210:LED_RGB_1210_with3DShape
- J1: footprint Connector_PinHeader_2.54mm:PinHeader_1x07_P2.54mm_Vertical -> Connector Custom:PinHeader_1x07_P2.54mm_Vertical
- renumbered CE to C3
