File: pcb/LP5012.kicad_pcb (KiCad board)
At the start: 2 copper layers, 16.2 x 24.5 mm, 16 parts, among them J1 Main Connector, U1 LP5012

Commit message: Inlcusión de notas de fabricación
Other:
- board text added: "Terminación superficial: HASL con plomo Grosor: 1.6mm Materíal: FR4 TG130-140 Color de Máscara de soldadura: Verde Color de Serigrafía: Blanco Mínimo ancho de pista: 0.2mm Mínimo diámetro de perforación: 0.5mm Grilla utilizada: 0.1mm"
Changed lines of the file:
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@@
   (general
     (thickness 1.6)
-    (drawings 16)
+    (drawings 17)
     (tracks 198)
     (zones 0)
@@
       (xy -4.235267 0.235728) (xy -4.090427 0.253706) (xy -4.00685 0.256255) (xy -3.873174 0.251818)) (layer B.SilkS) (width 0.01))
   )
+  (gr_text "Terminación superficial: HASL con plomo\nGrosor: 1.6mm\nMateríal: FR4 TG130-140\nColor de Máscara de soldadura: Verde\nColor de Serigrafía: Blanco\nMínimo ancho de pista: 0.2mm\nMínimo diámetro de perforación:  0.5mm\nGrilla utilizada: 0.1mm\n" (at 165.4 94.3) (layer F.Fab)
+    (effects (font (size 1 1) (thickness 0.15)) (justify left))
+  )
   (gr_text "Led Driver\nVersion 1.0" (at 148.2 91.7 270) (layer B.SilkS)
