File: pcb/LP5012.sch (KiCad schematic (older format))
At the start: 10 parts, among them J1 Main Connector, U1 LP5012

Commit message: Depuración de archivos sobrantes y estructuración de carpetas
Se añaden carpetas doc, info y pcb.
Se limpian archivos que estaban de más.
Parts:
- removed D3, D4: LED_RGB, LED_SMD:LED_RGB_5050-6, symbol Device:LED_RGB
- added D1, D2, D3, D4, D5, D6: LED, LED_SMD:LED_0805_2012Metric, symbol Device:LED
- D7: renamed from D1; footprint LED_SMD:LED_RGB_5050-6 -> LED_SMD:LED_RGB_1210; symbol Device:LED_RGB -> Device:LED_ABRG
- D8: renamed from D2; footprint LED_SMD:LED_RGB_5050-6 -> LED_SMD:LED_RGB_1210; symbol Device:LED_RGB -> Device:LED_ABRG
- U1: footprint Footprint LP5012:PQFN21P40_300X300X80L40X20T180 -> Footprint LP5012:LP5012; symbol LP5012_SCH:LP5012 -> LP5012:LP5012
Connections:
- wire segments 93 -> 85
Other:
- note added: "LEDs"
- note added: "Project Name: LP5012 Led Driver Module\nAuthor: Jhonattan Camargo"
- note added: "Via Layout Design from the chip manufacturer.\nPage 45: http://www.ti.com/lit/ds/symlink/lp5012.pdf\nrepo\doc\3. Huella recomendada.png\n"
- note removed: "Author: Jhonattan Camargo"
- note removed: "LEDs RGB"
- note removed: "Via Layout Design from the chip manufacturer.\nPage 45: http://www.ti.com/lit/ds/symlink/lp5012.pdf\n"
Changed lines of the file:
@@
 EESchema Schematic File Version 4
-LIBS:LP5012EVM_Custom-cache
 EELAYER 30 0
 EELAYER END
@@
 $EndComp
 $Comp
-L Device:LED_RGB D1
+L Device:LED_ABRG D7
 U 1 1 5D929F43
-P 9400 2300
-F 0 "D1" H 9350 2700 50  0000 C CNN
-F 1 "LED_RGB" H 9400 1950 50  0001 C CNN
-F 2 "LED_SMD:LED_RGB_5050-6" H 9400 2250 50  0001 C CNN
-F 3 "~" H 9400 2250 50  0001 C CNN
-	1    9400 2300
-	1    0    0    -1
-$EndComp
-$Comp
-L Device:LED_RGB D2
-U 1 1 5D92CB70
-P 9400 3250
-F 0 "D2" H 9350 3650 50  0000 C CNN
-F 1 "LED_RGB" H 9400 2900 50  0001 C CNN
-F 2 "LED_SMD:LED_RGB_5050-6" H 9400 3200 50  0001 C CNN
-F 3 "~" H 9400 3200 50  0001 C CNN
-	1    9400 3250
-	1    0    0    -1
-$EndComp
-$Comp
-L Device:LED_RGB D3
-U 1 1 5D92D562
 P 9400 4350
-F 0 "D3" H 9350 4750 50  0000 C CNN
+F 0 "D7" H 9350 4750 50  0000 C CNN
 F 1 "LED_RGB" H 9400 4000 50  0001 C CNN
-F 2 "LED_SMD:LED_RGB_5050-6" H 9400 4300 50  0001 C CNN
+F 2 "LED_SMD:LED_RGB_1210" H 9400 4300 50  0001 C CNN
 F 3 "~" H 9400 4300 50  0001 C CNN
 	1    9400 4350
@@
 $EndComp
 $Comp
-L Device:LED_RGB D4
-U 1 1 5D92EA6C
+L Device:LED_ABRG D8
+U 1 1 5D92CB70
 P 9400 5300
-F 0 "D4" H 9350 5700 50  0000 C CNN
+F 0 "D8" H 9350 5700 50  0000 C CNN
 F 1 "LED_RGB" H 9400 4950 50  0001 C CNN
-F 2 "LED_SMD:LED_RGB_5050-6" H 9400 5250 50  0001 C CNN
+F 2 "LED_SMD:LED_RGB_1210" H 9400 5250 50  0001 C CNN
 F 3 "~" H 9400 5250 50  0001 C CNN
 	1    9400 5300
@@
 LB9
 Wire Wire Line
-	9200 2100 9050 2100
-Wire Wire Line
-	9200 2300 9050 2300
-Wire Wire Line
-	9200 2500 9050 2500
-Wire Wire Line
-	9050 3050 9200 3050
-Wire Wire Line
-	9200 3250 9050 3250
-Wire Wire Line
-	9050 3450 9200 3450
-Wire Wire Line
 	9200 4150 9050 4150
 Wire Wire Line
-	9050 4350 9200 4350
+	9200 4350 9050 4350
 Wire Wire Line
 	9200 4550 9050 4550
 Wire Wire Line
 	9050 5100 9200 5100
+Wire Wire Line
+	9200 5300 9050 5300
 Wire Wire Line
 	9050 5500 9200 5500
 Text Label 9050 5500 2    50   ~ 0
 LB11
-Wire Wire Line
-	9200 5300 9050 5300
 Text Label 9050 5300 2    50   ~ 0
 LB10
@@
 20-09-2019
 $Comp
-L LP5012_SCH:LP5012 U1
+L LP5012:LP5012 U1
 U 1 1 5D99BF30
 P 6300 3300
 F 0 "U1" H 6000 3950 50  0000 C CNN
 F 1 "LP5012" H 6150 2050 50  0000 C CNN
-F 2 "Footprint LP5012:PQFN21P40_300X300X80L40X20T180" H 6250 3950 50  0001 C CNN
+F 2 "Footprint LP5012:LP5012" H 6250 3950 50  0001 C CNN
 F 3 "" H 6250 3950 50  0000 C CNN
 	1    6300 3300
@@
 Text Label 1350 3700 0    50   ~ 0
 IN_EN
-Text Label 1350 3800 0    50   ~ 0
-ADDR0
-Text Label 1350 3900 0    50   ~ 0
-ADDR1
 Wire Wire Line
 	1650 2850 1650 3150
@@
 	5700 4400 5700 4650
 Text Notes 5900 4800 0    50   ~ 0
-Via Layout Design from the chip manufacturer.\nPage 45: http://www.ti.com/lit/ds/symlink/lp5012.pdf\n
+Via Layout Design from the chip manufacturer.\nPage 45: http://www.ti.com/lit/ds/symlink/lp5012.pdf\nrepo\doc\3. Huella recomendada.png\n
 Wire Wire Line
 	4550 2800 5850 2800
@@
 Wire Wire Line
 	1350 3700 1750 3700
-Wire Wire Line
-	1750 3800 1350 3800
 Wire Wire Line
 	1750 3900 1350 3900
@@
 L power:VCC #PWR0107
 U 1 1 5D98000B
+P 9900 4000
+F 0 "#PWR0107" H 9900 3850 50  0001 C CNN
+F 1 "VCC" H 9917 4173 50  0000 C CNN
+F 2 "" H 9900 4000 50  0001 C CNN
+F 3 "" H 9900 4000 50  0001 C CNN
+	1    9900 4000
+	1    0    0    -1
+$EndComp
+$Comp
+L power:VCC #PWR0110
+U 1 1 5D981315
+P 9900 4950
+F 0 "#PWR0110" H 9900 4800 50  0001 C CNN
+F 1 "VCC" H 9917 5123 50  0000 C CNN
+F 2 "" H 9900 4950 50  0001 C CNN
+F 3 "" H 9900 4950 50  0001 C CNN
+	1    9900 4950
+	1    0    0    -1
+$EndComp
+$Comp
+L power:VCC #PWR0111
+U 1 1 5D981A4D
 P 9900 1950
-F 0 "#PWR0107" H 9900 1800 50  0001 C CNN
+F 0 "#PWR0111" H 9900 1800 50  0001 C CNN
 F 1 "VCC" H 9917 2123 50  0000 C CNN
 F 2 "" H 9900 1950 50  0001 C CNN
@@
 $EndComp
 $Comp
-L power:VCC #PWR0110
-U 1 1 5D981315
-P 9900 2900
-F 0 "#PWR0110" H 9900 2750 50  0001 C CNN
-F 1 "VCC" H 9917 3073 50  0000 C CNN
-F 2 "" H 9900 2900 50  0001 C CNN
-F 3 "" H 9900 2900 50  0001 C CNN
-	1    9900 2900
-	1    0    0    -1
-$EndComp
-$Comp
-L power:VCC #PWR0111
-U 1 1 5D981A4D
-P 9900 4000
-F 0 "#PWR0111" H 9900 3850 50  0001 C CNN
-F 1 "VCC" H 9917 4173 50  0000 C CNN
-F 2 "" H 9900 4000 50  0001 C CNN
-F 3 "" H 9900 4000 50  0001 C CNN
-	1    9900 4000
-	1    0    0    -1
-$EndComp
-$Comp
 L power:VCC #PWR0112
 U 1 1 5D981FA3
-P 9950 4950
-F 0 "#PWR0112" H 9950 4800 50  0001 C CNN
-F 1 "VCC" H 9967 5123 50  0000 C CNN
-F 2 "" H 9950 4950 50  0001 C CNN
-F 3 "" H 9950 4950 50  0001 C CNN
-	1    9950 4950
-	1    0    0    -1
-$EndComp
+P 9950 2900
+F 0 "#PWR0112" H 9950 2750 50  0001 C CNN
+F 1 "VCC" H 9967 3073 50  0000 C CNN
+F 2 "" H 9950 2900 50  0001 C CNN
+F 3 "" H 9950 2900 50  0001 C CNN
+	1    9950 2900
+	1    0    0    -1
+$EndComp
+Wire Wire Line
+	9600 5300 9900 5300
 Wire Wire Line
 	9900 2500 9900 2300
-Wire Wire Line
-	9600 2500 9900 2500
 Connection ~ 9900 2100
 Wire Wire Line
 	9900 2100 9900 1950
-Wire Wire Line
-	9600 2100 9900 2100
 Connection ~ 9900 2300
 Wire Wire Line
 	9900 2300 9900 2100
 Wire Wire Line
-	9900 3450 9900 3250
-Wire Wire Line
-	9600 3450 9900 3450
-Wire Wire Line
-	9600 3050 9900 3050
-Connection ~ 9900 3050
-Wire Wire Line
-	9900 3050 9900 2900
-Wire Wire Line
-	9600 3250 9900 3250
-Connection ~ 9900 3250
-Wire Wire Line
-	9900 3250 9900 3050
-Wire Wire Line
-	9900 4550 9900 4350
-Wire Wire Line
-	9600 4550 9900 4550
-Wire Wire Line
-	9600 4150 9900 4150
-Connection ~ 9900 4150
-Wire Wire Line
-	9900 4150 9900 4000
+	9950 3450 9950 3250
+Connection ~ 9950 3050
+Wire Wire Line
+	9950 3050 9950 2900
+Connection ~ 9950 3250
+Wire Wire Line
+	9950 3250 9950 3050
 Wire Wire Line
 	9600 4350 9900 4350
-Connection ~ 9900 4350
-Wire Wire Line
-	9900 4350 9900 4150
-Wire Wire Line
-	9950 5500 9950 5300
-Wire Wire Line
-	9600 5500 9950 5500
-Wire Wire Line
-	9600 5100 9950 5100
-Connection ~ 9950 5100
-Wire Wire Line
-	9950 5100 9950 4950
-Wire Wire Line
-	9600 5300 9950 5300
-Connection ~ 9950 5300
-Wire Wire Line
-	9950 5300 9950 5100
-Wire Wire Line
-	9600 2300 9900 2300
 Wire Notes Line
 	950  2400 3400 2400
@@
 LED Driver IC
 Text Notes 8700 6000 0    98   ~ 0
-LEDs RGB
-Text Notes 7000 6950 0    98   ~ 0
-Author: Jhonattan Camargo
+LEDs
 Text Label 1350 3600 0    50   ~ 0
 SDA
 Text Label 1350 3500 0    50   ~ 0
 SCL
+$Comp
+L Device:LED D1
+U 1 1 5D9A8567
+P 9400 2100
+F 0 "D1" H 9550 2200 50  0000 C CNN
+F 1 "LED" H 9393 2225 50  0001 C CNN
+F 2 "LED_SMD:LED_0805_2012Metric" H 9400 2100 50  0001 C CNN
+F 3 "~" H 9400 2100 50  0001 C CNN
+	1    9400 2100
+	1    0    0    -1
+$EndComp
+$Comp
+L Device:LED D2
+U 1 1 5D9A9184
+P 9400 2300
+F 0 "D2" H 9550 2400 50  0000 C CNN
+F 1 "LED" H 9393 2425 50  0001 C CNN
+F 2 "LED_SMD:LED_0805_2012Metric" H 9400 2300 50  0001 C CNN
+F 3 "~" H 9400 2300 50  0001 C CNN
+	1    9400 2300
+	1    0    0    -1
+$EndComp
+$Comp
+L Device:LED D3
+U 1 1 5D9A955B
+P 9400 2500
+F 0 "D3" H 9550 2600 50  0000 C CNN
+F 1 "LED" H 9393 2625 50  0001 C CNN
+F 2 "LED_SMD:LED_0805_2012Metric" H 9400 2500 50  0001 C CNN
+F 3 "~" H 9400 2500 50  0001 C CNN
+	1    9400 2500
+	1    0    0    -1
+$EndComp
+$Comp
+L Device:LED D4
+U 1 1 5D9A9A6A
+P 9400 3050
+F 0 "D4" H 9550 3150 50  0000 C CNN
+F 1 "LED" H 9393 3175 50  0001 C CNN
+F 2 "LED_SMD:LED_0805_2012Metric" H 9400 3050 50  0001 C CNN
+F 3 "~" H 9400 3050 50  0001 C CNN
+	1    9400 3050
+	1    0    0    -1
+$EndComp
+$Comp
+L Device:LED D5
+U 1 1 5D9AA001
+P 9400 3250
+F 0 "D5" H 9550 3350 50  0000 C CNN
+F 1 "LED" H 9393 3375 50  0001 C CNN
+F 2 "LED_SMD:LED_0805_2012Metric" H 9400 3250 50  0001 C CNN
+F 3 "~" H 9400 3250 50  0001 C CNN
+	1    9400 3250
+	1    0    0    -1
+$EndComp
+$Comp
+L Device:LED D6
+U 1 1 5D9AA1F8
+P 9400 3450
+F 0 "D6" H 9550 3550 50  0000 C CNN
+F 1 "LED" H 9393 3575 50  0001 C CNN
+F 2 "LED_SMD:LED_0805_2012Metric" H 9400 3450 50  0001 C CNN
+F 3 "~" H 9400 3450 50  0001 C CNN
+	1    9400 3450
+	1    0    0    -1
+$EndComp
+Wire Wire Line
+	9050 2100 9250 2100
+Wire Wire Line
+	9050 2300 9250 2300
+Wire Wire Line
+	9550 2100 9900 2100
+Wire Wire Line
+	9550 2300 9900 2300
+Wire Wire Line
+	9050 2500 9250 2500
+Wire Wire Line
+	9550 2500 9900 2500
+Wire Wire Line
+	9050 3050 9250 3050
+Wire Wire Line
+	9050 3250 9250 3250
+Wire Wire Line
+	9050 3450 9250 3450
+Wire Wire Line
+	9550 3450 9950 3450
+Wire Wire Line
+	9550 3250 9950 3250
+Wire Wire Line
+	9550 3050 9950 3050
+Wire Wire Line
+	9900 4950 9900 5300
+Wire Wire Line
+	9900 4000 9900 4350
+Text Notes 7000 7000 0    118  ~ 0
+Project Name: LP5012 Led Driver Module\nAuthor: Jhonattan Camargo
+Text Label 1350 3800 0    50   ~ 0
+ADDR1
+Wire Wire Line
+	1750 3800 1350 3800
+Text Label 1350 3900 0    50   ~ 0
+ADDR0
 $EndSCHEMATC

Commit message: Inclusión de modelos 3D y modificación de algunas liberías
Parts:
- D7, D8: footprint LED_SMD:LED_RGB_1210 -> LED_RGB_1210:LED_RGB_1210_with3DShape
- J1: footprint Connector_PinHeader_2.54mm:PinHeader_1x07_P2.54mm_Vertical -> Connector Custom:PinHeader_1x07_P2.54mm_Vertical
Changed lines of the file:
@@
 F 0 "D7" H 9350 4750 50  0000 C CNN
 F 1 "LED_RGB" H 9400 4000 50  0001 C CNN
-F 2 "LED_SMD:LED_RGB_1210" H 9400 4300 50  0001 C CNN
+F 2 "LED_RGB_1210:LED_RGB_1210_with3DShape" H 9400 4300 50  0001 C CNN
 F 3 "~" H 9400 4300 50  0001 C CNN
 	1    9400 4350
@@
 F 0 "D8" H 9350 5700 50  0000 C CNN
 F 1 "LED_RGB" H 9400 4950 50  0001 C CNN
-F 2 "LED_SMD:LED_RGB_1210" H 9400 5250 50  0001 C CNN
+F 2 "LED_RGB_1210:LED_RGB_1210_with3DShape" H 9400 5250 50  0001 C CNN
 F 3 "~" H 9400 5250 50  0001 C CNN
 	1    9400 5300
@@
 F 0 "J1" H 2030 3642 50  0000 L CNN
 F 1 "Main Connector" H 2030 3551 50  0001 L CNN
-F 2 "Connector_PinHeader_2.54mm:PinHeader_1x07_P2.54mm_Vertical" H 1950 3600 50  0001 C CNN
+F 2 "Connector Custom:PinHeader_1x07_P2.54mm_Vertical" H 1950 3600 50  0001 C CNN
 F 3 "~" H 1950 3600 50  0001 C CNN
 	1    1950 3600

Commit message: Inclusión de cambios de revisión 2
Connections:
- net LB0 renamed LED0
- net LB1 renamed LED1
- net LB10 renamed LED10
- net LB11 renamed LED11
- net LB2 renamed LED2
- net LB3 renamed LED3
- net LB4 renamed LED4
- net LB5 renamed LED5
- net LB6 renamed LED6
- net LB7 renamed LED7
- net LB8 renamed LED8
- net LB9 renamed LED9
Other:
- note added: "ISET = 73.5/R4"
- note added: "ISET(10k) = 7.35mA"
- note added: "ISET(3.3k) = 22.3mA"
- note added: "VCC Range: 2.7V to 5.5V\nICC Max Range: ISET * 12\nIt's expected that the host include the pull-up resistors."
- note removed: "Iset = 73.5/R4"
- note removed: "Iset(3.3k) = 22.3mA"
- note removed: "It's expected that the host include the pull-up resistors"
- note removed: "Project Name: LP5012 Led Driver Module\nAuthor: Jhonattan Camargo"
- moved on the sheet: D1, D2, D3, D4, D5, D6, D7, D8, J1

Commit message: Ultimas modificaciones
Parts:
- C2, C3: Link (none) -> https://ar.mouser.com/ProductDetail/KEMET/C0805C105K3RACTU?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; SKU (none) -> 80-C0805C105K3R; Supplier (none) -> Mouser
- C4: Link (none) -> https://ar.mouser.com/ProductDetail/KEMET/C0805C104J5RACTU?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; SKU (none) -> 80-C0805C104J5R; Supplier (none) -> Mouser
- D1, D2, D3, D4, D5, D6: Link (none) -> https://ar.mouser.com/ProductDetail/Inolux/IN-S85ATG?qs=sGA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; SKU (none) -> 743-IN-S85ATG; Supplier (none) -> Mouser
- D7, D8: Link (none) -> 638-19237R6GHBHCA01; SKU (none) -> 638-19237R6GHBHCA01; Supplier (none) -> Mouser
- R4: Link (none) -> https://ar.mouser.com/ProductDetail/Vishay-Dale/CRCW08053K3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; SKU (none) -> 71-CRCW08053K30FKEAC; Supplier (none) -> Mouser
- U1: Link (none) -> https://ar.mouser.com/ProductDetail/Texas-Instruments/LP501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; SKU (none) -> 595-LP5012RUKR; Supplier (none) -> Mouser
